File: splitflappcb.kicad_sch (KiCad schematic)
At the start: 42 parts, among them J1 Conn_01x04_Pin, J2 Conn_01x04_Pin, J3 Conn_01x05_Pin, J4 AddressJumpers, J5 HallSensor, J6 AVR-ISP-6, J7 Serial-328P, J8 Serial-ESP12E, J9 WS2815, SW1 RESET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

Commit message: update to rev1.1
Parts:
- added R8: 10k, Resistor_SMD:R_0402_1005Metric, symbol Device:R_Small
Connections:
- net GND: now also R8.2
- net at U4.16 (GPIO15): now also R8.1
Changed lines of the file:
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@@
   (junction (at 116.84 153.67) (diameter 0) (color 0 0 0 0)
   )
+  (junction (at 233.68 151.13) (diameter 0) (color 0 0 0 0)
+  )
   (junction (at 97.79 134.62) (diameter 0) (color 0 0 0 0)
   )
@@
     (stroke (width 0) (type default))
   )
+  (wire (pts (xy 256.54 147.32) (xy 256.54 151.13))
+    (stroke (width 0) (type default))
+  )
   (wire (pts (xy 33.02 46.99) (xy 49.53 46.99))
     (stroke (width 0) (type default))
@@
     (stroke (width 0) (type default))
   )
+  (wire (pts (xy 256.54 151.13) (xy 233.68 151.13))
+    (stroke (width 0) (type default))
+  )
   (wire (pts (xy 248.92 71.12) (xy 255.27 71.12))
     (stroke (width 0) (type default))
   )
+  (wire (pts (xy 233.68 151.13) (xy 233.68 152.4))
+    (stroke (width 0) (type default))
+  )
   (wire (pts (xy 166.37 54.61) (xy 176.53 54.61))
     (stroke (width 0) (type default))
@@
     (stroke (width 0) (type default))
   )
+  (wire (pts (xy 248.92 139.7) (xy 256.54 139.7))
+    (stroke (width 0) (type default))
+  )
   (wire (pts (xy 64.77 64.77) (xy 67.31 64.77))
     (stroke (width 0) (type default))
@@
     (stroke (width 0) (type default))
   )
+  (wire (pts (xy 256.54 139.7) (xy 256.54 142.24))
+    (stroke (width 0) (type default))
+  )
   (wire (pts (xy 92.71 133.35) (xy 92.71 134.62))
     (stroke (width 0) (type default))
@@
     (stroke (width 0) (type default))
   )
-  (wire (pts (xy 233.68 149.86) (xy 233.68 152.4))
+  (wire (pts (xy 233.68 149.86) (xy 233.68 151.13))
     (stroke (width 0) (type default))
   )
@@
         )
       )
+    )
+  )
+  (symbol (lib_id "Device:R_Small") (at 256.54 144.78 0) (mirror y) (unit 1)
+    (in_bom yes) (on_board yes) (dnp no)
+    (property "Reference" "R8" (at 260.35 143.51 0)
+      (effects (font (size 1.27 1.27)))
+    )
+    (property "Value" "10k" (at 260.35 146.05 0)
+      (effects (font (size 1.27 1.27)))
+    )
+    (property "Footprint" "Resistor_SMD:R_0402_1005Metric" (at 256.54 144.78 0)
+      (effects (font (size 1.27 1.27)) hide)
+    )
+    (property "Datasheet" "~" (at 256.54 144.78 0)
+      (effects (font (size 1.27 1.27)) hide)
+    )
+    (property "LCSC" "C25744" (at 256.54 144.78 0)
+      (effects (font (size 1.27 1.27)) hide)
+    )
+    (pin "1")
+    (pin "2")
+    (instances
+      (project "splitflappcb"
+        (path "/3e6df37b-d512-4c66-98b7-ac402904e438"
+          (reference "R8") (unit 1)
+        )
+      )
